File: PCB/macro_pad.kicad_pcb (KiCad board)
At the start: 2 copper layers, 43 parts, among them J1 Conn_01x04_Pin, SW1 SW_Push_45deg, SW10 SW_Push_45deg, SW11 SW_Push_45deg, SW12 SW_Push_45deg, SW13 RotaryEncoder, SW2 SW_Push_45deg, SW3 SW_Push_45deg, SW4 SW_Push_45deg, SW5 SW_Push_45deg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

Commit message: Started laying out PCB
Parts:
- removed D10, D12, D14, D16: SK6812MINI, LED_SMD:LED_SK6812MINI_PLCC4_3.5x3.5mm_P1.75mm
- D17, D18, D19, D20, D21, D22, D23, D24, D29, D30, D31, D32: moved to B.Cu
- moved J1 73.7 mm to (55.9, 23.7)
- moved SW13 68.7 mm to (127.7, 26.1)
- moved D17 67.4 mm to (85.0, 107.6), turned to -90 degrees
- moved D18 63.3 mm to (88.5, 107.6), turned to -90 degrees
- moved D19 59.4 mm to (92.0, 107.6), turned to -90 degrees
- moved U1 57.6 mm to (109.2, 29.8)
- moved D20 55.7 mm to (95.6, 107.6), turned to -90 degrees
- moved D21 52.2 mm to (99.2, 107.6), turned to -90 degrees
- moved D22 49.0 mm to (102.7, 107.6), turned to -90 degrees
- moved D4 46.8 mm to (96.0, 62.7)
- moved D23 46.1 mm to (106.2, 107.6), turned to -90 degrees
- moved D1 43.8 mm to (76.7, 62.9)
- moved D24 43.5 mm to (109.8, 107.6), turned to -90 degrees
- moved D11 41.5 mm to (134.2, 62.6)
- moved D29 41.5 mm to (113.3, 107.6), turned to -90 degrees
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Connections:
- D15 pad 1: Net-(D10-DIN) -> unconnected-(D15-DOUT-Pad1)
- J1 pad 1: unconnected-(J1-Pin_1-Pad1) -> GND
- J1 pad 2: unconnected-(J1-Pin_2-Pad2) -> +3.3V
- U1 pad 12: unconnected-(U1-3V3-Pad12) -> +3.3V
Other:
- board outline added: 100 x 99.8 mm

Commit message: Got the traces routed
Routing:
- net GND: track 0.00 -> 305.3 mm, vias 0 -> 3
- net +5V: track 0.00 -> 259.9 mm, vias 0 -> 3
- net Row 3: track 0.00 -> 116.9 mm
- net Net-(D29-A): track 0.00 -> 106.3 mm, vias 0 -> 1
- net Row 2: track 0.00 -> 106.1 mm
- net Row 1: track 0.00 -> 95.6 mm
- net Col 2: track 0.00 -> 95.6 mm
- net Col 3: track 0.00 -> 82.3 mm, vias 0 -> 1
- net Net-(D32-A): track 0.00 -> 77.9 mm, vias 0 -> 2
- net Col 4: track 0.00 -> 77.8 mm
- net Net-(D3-DOUT): track 0.00 -> 77.0 mm, vias 0 -> 2
- net Net-(D17-A): track 0.00 -> 71.4 mm, vias 0 -> 1
- net Net-(D31-A): track 0.00 -> 70.5 mm
- net Net-(D20-A): track 0.00 -> 68.6 mm
- net Col 1: track 0.00 -> 65.8 mm, vias 0 -> 1
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Other:
- board text added: "XIAO HERE"

Commit message: adding silk screen and created the gerbers
Other:
- board text added: "Minecraftchest2 macro pad"
