File: PCB/macro_pad.kicad_sch (KiCad schematic)
At the start: 39 parts, among them J1 Conn_01x04_Pin, SW1 SW_Push_45deg, SW10 SW_Push_45deg, SW11 SW_Push_45deg, SW12 SW_Push_45deg, SW13 RotaryEncoder, SW2 SW_Push_45deg, SW3 SW_Push_45deg, SW4 SW_Push_45deg, SW5 SW_Push_45deg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

Commit message: Got the case for the PCB made
Parts:
- removed D1, D11, D13, D15, D2, D3, D4, D5, D6, D7, D8, D9: SK6812MINI, LED_SMD:LED_SK6812MINI_PLCC4_3.5x3.5mm_P1.75mm, symbol LED:SK6812MINI
- removed D17, D18, D19: 1N4148, Diode_THT:D_DO-35_SOD27_P7.62mm_Horizontal, symbol Diode:1N4148
- added D1, D2, D3: 1N4148, Diode_THT:D_DO-35_SOD27_P7.62mm_Horizontal, symbol Diode:1N4148
- SW1, SW10, SW11, SW12, SW2, SW3, SW4, SW5, SW6, SW7, SW8, SW9: footprint mx-sold:MX-Solderable-1U -> Button_Switch_Keyboard:SW_Cherry_MX_1.00u_PCB
Connections:
- net LED Data is gone; now on net Col 4: U1.11 (GPIO3/MOSI)
- net Col 1: now also SW1.2, SW4.2, U1.3 (GPIO28/ADC2/A2); no longer SW8.2, SW9.2, U1.5 (GPIO6/SDA)
- net Col 2: now also SW2.2, SW5.2, SW8.2, U1.4 (GPIO29/ADC3/A3); no longer SW10.2, SW4.2, SW6.2, U1.6 (GPIO7/SCL)
- net Col 3: now also SW3.2, SW6.2, SW9.2; no longer SW1.2, SW11.2, SW5.2
- net Col 4: now also SW10.2, SW11.2; no longer SW2.2, SW3.2
- net OLED SCL: now also U1.6 (GPIO7/SCL); no longer U1.3 (GPIO28/ADC2/A2)
- net OLED SDA: now also U1.5 (GPIO6/SDA); no longer U1.4 (GPIO29/ADC3/A3)
- net Row 1: now also D1.1 (K)
- net Row 2: now also D2.1 (K)
- net Row 3: now also D3.1 (K)
- net at D24.2 (A): now also SW5.1; no longer SW6.1
- net at D30.2 (A): now also SW9.1; no longer SW11.1
- net at SW8.1: now also D31.2 (A); no longer D21.2 (A)
- net at D20.2 (A): now also SW3.1; no longer SW5.1
- net at SW10.1: now also D1.2 (A); no longer D31.2 (A)
- net at SW4.1: now also D22.2 (A); no longer D23.2 (A)
- net at D29.2 (A): now also SW6.1; no longer SW1.1
- net at SW12.1: now also D3.2 (A)
- net at D32.2 (A): now also SW7.1; no longer SW9.1
- net at SW2.1: now also D23.2 (A)
- new net: D2.2 (A), SW11.1
- new net: D21.2 (A), SW1.1
